Commit message: processed ucb dataset, update grasp generation

File: assets/allegro/allegro.urdf (robot description, URDF)
Before this commit: robot allegro_hand_right, 21 links, 20 joints
Links:
- link base_link: geometry collision box size=0.0408 0.1130 0.095; visual mesh filename=allegro/meshes/allegro/base_link.obj
